File: ecad/shockboard/shockboard.kicad_pcb (KiCad board)
At the start: 2 copper layers, 0 parts

Commit message: Added new kicad file format and preliminary ergogen layout
Other:
- net class Default removed
