File: ergogen/shockboard-v0_4_0/output/pcbs/shockboard.kicad_pcb (KiCad board)
At the start: 2 copper layers, 295.7 x 128.2 mm, 105 parts

Commit message: feat: corrected nets for rows and columns
Connections:
- D1 pad 2: (no net) -> P7
- D10 pad 2: (no net) -> P8
- D11 pad 2: (no net) -> P9
- D12 pad 2: (no net) -> P6
- D13 pad 2: (no net) -> P7
- D14 pad 2: (no net) -> P8
- D15 pad 2: (no net) -> P9
- D16 pad 2: (no net) -> P6
- D17 pad 2: (no net) -> P7
- D18 pad 2: (no net) -> P8
- D19 pad 2: (no net) -> P9
- D2 pad 2: (no net) -> P8
- D20 pad 2: (no net) -> P6
- D21 pad 2: (no net) -> P7
- D22 pad 2: (no net) -> P8
- D23 pad 2: (no net) -> P9
- D24 pad 2: (no net) -> P16
- D25 pad 2: (no net) -> P16
- D26 pad 2: (no net) -> P16
- D27 pad 2: (no net) -> P7
- D28 pad 2: (no net) -> P8
- D29 pad 2: (no net) -> P9
- D3 pad 2: (no net) -> P9
- D30 pad 2: (no net) -> P6
- D31 pad 2: (no net) -> P7
- D32 pad 2: (no net) -> P8
- D33 pad 2: (no net) -> P9
- D34 pad 2: (no net) -> P6
- D35 pad 2: (no net) -> P7
- D36 pad 2: (no net) -> P8
- D37 pad 2: (no net) -> P9
- D38 pad 2: (no net) -> P6
- D39 pad 2: (no net) -> P7
- D4 pad 2: (no net) -> P6
- D40 pad 2: (no net) -> P8
- D41 pad 2: (no net) -> P9
- D42 pad 2: (no net) -> P6
- D43 pad 2: (no net) -> P7
- D44 pad 2: (no net) -> P8
- D45 pad 2: (no net) -> P9
- D46 pad 2: (no net) -> P6
- D47 pad 2: (no net) -> P7
- D48 pad 2: (no net) -> P8
- D49 pad 2: (no net) -> P9
- D5 pad 2: (no net) -> P7
- D50 pad 2: (no net) -> P16
- D51 pad 2: (no net) -> P16
- D52 pad 2: (no net) -> P16
- D6 pad 2: (no net) -> P8
- D7 pad 2: (no net) -> P9
- D8 pad 2: (no net) -> P6
- D9 pad 2: (no net) -> P7
- S1 pad 1: (no net) -> P7
- S1 pad 2: P0 -> P1
- S10 pad 1: (no net) -> P8
- S11 pad 1: (no net) -> P9
- S12 pad 1: (no net) -> P6
- S13 pad 1: (no net) -> P7
- S14 pad 1: (no net) -> P8
- S15 pad 1: (no net) -> P9
- S16 pad 1: (no net) -> P6
- S17 pad 1: (no net) -> P7
- S18 pad 1: (no net) -> P8
- S19 pad 1: (no net) -> P9
- S2 pad 1: (no net) -> P8
- S2 pad 2: P0 -> P1
- S20 pad 1: (no net) -> P6
- S21 pad 1: (no net) -> P7
- S22 pad 1: (no net) -> P8
- S23 pad 1: (no net) -> P9
- S24 pad 1: (no net) -> P16
- S25 pad 1: (no net) -> P16
- S26 pad 1: (no net) -> P16
- S27 pad 1: (no net) -> P7
- S27 pad 2: P11 -> P21
- S28 pad 1: (no net) -> P8
- S28 pad 2: P11 -> P21
- S29 pad 1: (no net) -> P9
- S29 pad 2: P11 -> P21
- S3 pad 1: (no net) -> P9
- S3 pad 2: P0 -> P1
- S30 pad 1: (no net) -> P6
- S30 pad 2: P10 -> P20
- S31 pad 1: (no net) -> P7
- S31 pad 2: P10 -> P20
- S32 pad 1: (no net) -> P8
- S32 pad 2: P10 -> P20
- S33 pad 1: (no net) -> P9
- S33 pad 2: P10 -> P20
- S34 pad 1: (no net) -> P6
- S34 pad 2: P9 -> P19
- S35 pad 1: (no net) -> P7
- S35 pad 2: P9 -> P19
- S36 pad 1: (no net) -> P8
- S36 pad 2: P9 -> P19
- S37 pad 1: (no net) -> P9
- S37 pad 2: P9 -> P19
- S38 pad 1: (no net) -> P6
- S38 pad 2: P8 -> P18
- S39 pad 1: (no net) -> P7
- S39 pad 2: P8 -> P18
- S4 pad 1: (no net) -> P6
- S4 pad 2: P1 -> P0
- S40 pad 1: (no net) -> P8
- S40 pad 2: P8 -> P18
- S41 pad 1: (no net) -> P9
- S41 pad 2: P8 -> P18
- S42 pad 1: (no net) -> P6
- S42 pad 2: P7 -> P15
- S43 pad 1: (no net) -> P7
- S43 pad 2: P7 -> P15
- S44 pad 1: (no net) -> P8
- S44 pad 2: P7 -> P15
- S45 pad 1: (no net) -> P9
- S45 pad 2: P7 -> P15
- S46 pad 1: (no net) -> P6
- S46 pad 2: P6 -> P14
- S47 pad 1: (no net) -> P7
- S47 pad 2: P6 -> P14
- S48 pad 1: (no net) -> P8
- S48 pad 2: P6 -> P14
- S49 pad 1: (no net) -> P9
- S49 pad 2: P6 -> P14
- S5 pad 1: (no net) -> P7
- S5 pad 2: P1 -> P0
- S50 pad 1: (no net) -> P16
- S50 pad 2: P8 -> P18
- S51 pad 1: (no net) -> P16
- S51 pad 2: P7 -> P15
- S52 pad 1: (no net) -> P16
- S52 pad 2: P6 -> P14
- S6 pad 1: (no net) -> P8
- S6 pad 2: P1 -> P0
- S7 pad 1: (no net) -> P9
- S7 pad 2: P1 -> P0
- S8 pad 1: (no net) -> P6
- S9 pad 1: (no net) -> P7

Commit message: feat: added choc hotswap and battery connector
Parts:
- added PAD1: , SMDPad, F.Cu at (132.4, -66.1)
- added PAD2: , SMDPad, F.Cu at (132.4, -63.1)
- added S100: , PG1350, F.Cu at (162.5, -31.3)
- added S101: , PG1350, F.Cu at (159.9, -50.2)
- added S102: , PG1350, F.Cu at (208.2, 20.4)
- added S103: , PG1350, F.Cu at (180.0, 24.4)
- added S104: , PG1350, F.Cu at (151.9, 33.9)
- added S53: , PG1350, F.Cu at (2.64, -18.8)
- added S54: , PG1350, F.Cu at (5.29, -37.6)
- added S55: , PG1350, F.Cu at (7.93, -56.4)
- added S56: , PG1350, F.Cu at (18.8, 2.64)
- added S57: , PG1350, F.Cu at (21.5, -16.2)
- added S58: , PG1350, F.Cu at (24.1, -35.0)
- added S59: , PG1350, F.Cu at (26.7, -53.8)
- added S60: , PG1350, F.Cu at (39.1, -5.11)
- added S61: , PG1350, F.Cu at (41.7, -23.9)
- added S62: , PG1350, F.Cu at (44.4, -42.7)
- added S63: , PG1350, F.Cu at (47.0, -61.6)
- added S64: , PG1350, F.Cu at (58.3, -5.44)
- added S65: , PG1350, F.Cu at (61.0, -24.3)
- added S66: , PG1350, F.Cu at (63.6, -43.1)
- added S67: , PG1350, F.Cu at (66.3, -61.9)
- added S68: , PG1350, F.Cu at (76.4, 2.16)
- added S69: , PG1350, F.Cu at (79.1, -16.7)
- added S70: , PG1350, F.Cu at (81.7, -35.5)
- added S71: , PG1350, F.Cu at (84.4, -54.3)
- added S72: , PG1350, F.Cu at (95.0, 6.29)
- added S73: , PG1350, F.Cu at (97.7, -12.5)
- added S74: , PG1350, F.Cu at (100.3, -31.3)
- added S75: , PG1350, F.Cu at (103.0, -50.2)
- added S76: , PG1350, F.Cu at (54.7, 20.4)
- added S77: , PG1350, F.Cu at (82.9, 24.4)
- added S78: , PG1350, F.Cu at (111.0, 33.9)
- added S79: , PG1350, F.Cu at (260.2, -18.8)
- added S80: , PG1350, F.Cu at (257.6, -37.6)
- added S81: , PG1350, F.Cu at (255.0, -56.4)
- added S82: , PG1350, F.Cu at (244.1, 2.64)
- added S83: , PG1350, F.Cu at (241.4, -16.2)
- added S84: , PG1350, F.Cu at (238.8, -35.0)
- added S85: , PG1350, F.Cu at (236.1, -53.8)
- added S86: , PG1350, F.Cu at (223.8, -5.11)
- added S87: , PG1350, F.Cu at (221.2, -23.9)
- added S88: , PG1350, F.Cu at (218.5, -42.7)
- added S89: , PG1350, F.Cu at (215.9, -61.6)
- added S90: , PG1350, F.Cu at (204.6, -5.44)
- added S91: , PG1350, F.Cu at (201.9, -24.3)
- added S92: , PG1350, F.Cu at (199.3, -43.1)
- added S93: , PG1350, F.Cu at (196.6, -61.9)
- added S94: , PG1350, F.Cu at (186.4, 2.16)
- added S95: , PG1350, F.Cu at (183.8, -16.7)
- added S96: , PG1350, F.Cu at (181.2, -35.5)
- added S97: , PG1350, F.Cu at (178.5, -54.3)
- added S98: , PG1350, F.Cu at (167.8, 6.29)
- added S99: , PG1350, F.Cu at (165.2, -12.5)
- moved MCU1 1.25 mm to (131.4, -56.1)
Connections:
- S1 pad 2: P1 -> P21
- S10 pad 2: P2 -> P19
- S11 pad 2: P2 -> P19
- S12 pad 2: P3 -> P18
- S13 pad 2: P3 -> P18
- S14 pad 2: P3 -> P18
- S15 pad 2: P3 -> P18
- S16 pad 2: P4 -> P15
- S17 pad 2: P4 -> P15
- S18 pad 2: P4 -> P15
- S19 pad 2: P4 -> P15
- S2 pad 2: P1 -> P21
- S20 pad 2: P5 -> P14
- S21 pad 2: P5 -> P14
- S22 pad 2: P5 -> P14
- S23 pad 2: P5 -> P14
- S24 pad 2: P3 -> P18
- S25 pad 2: P4 -> P15
- S26 pad 2: P5 -> P14
- S27 pad 2: P21 -> P1
- S28 pad 2: P21 -> P1
- S29 pad 2: P21 -> P1
- S3 pad 2: P1 -> P21
- S30 pad 2: P20 -> P0
- S31 pad 2: P20 -> P0
- S32 pad 2: P20 -> P0
- S33 pad 2: P20 -> P0
- S34 pad 2: P19 -> P2
- S35 pad 2: P19 -> P2
- S36 pad 2: P19 -> P2
- S37 pad 2: P19 -> P2
- S38 pad 2: P18 -> P3
- S39 pad 2: P18 -> P3
- S4 pad 2: P0 -> P20
- S40 pad 2: P18 -> P3
- S41 pad 2: P18 -> P3
- S42 pad 2: P15 -> P4
- S43 pad 2: P15 -> P4
- S44 pad 2: P15 -> P4
- S45 pad 2: P15 -> P4
- S46 pad 2: P14 -> P5
- S47 pad 2: P14 -> P5
- S48 pad 2: P14 -> P5
- S49 pad 2: P14 -> P5
- S5 pad 2: P0 -> P20
- S50 pad 2: P18 -> P3
- S51 pad 2: P15 -> P4
- S52 pad 2: P14 -> P5
- S6 pad 2: P0 -> P20
- S7 pad 2: P0 -> P20
- S8 pad 2: P2 -> P19
- S9 pad 2: P2 -> P19

Commit message: wip: outline redesign
Parts:
- moved MCU1 181.7 mm to (212.4, 106.6)
- moved PAD1 181.7 mm to (213.4, 96.6)
- moved PAD2 181.7 mm to (213.4, 99.6)
- moved D26 164.0 mm to (189.7, 180.7)
- moved S24 164.0 mm to (135.6, 163.1)
- moved S26 164.0 mm to (191.9, 176.6)
- moved S76 164.0 mm to (135.6, 163.1)
- moved S78 164.0 mm to (191.9, 176.6)
- moved D24 164.0 mm to (138.5, 166.8)
- moved D4 164.0 mm to (99.1, 150.0)
- moved S4 164.0 mm to (99.7, 145.3)
- moved S56 164.0 mm to (99.7, 145.3)
- moved D12 164.0 mm to (138.6, 141.9)
- moved D13 164.0 mm to (141.2, 123.1)
- moved D38 164.0 mm to (286.2, 141.9)
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Connections:
- S1 pad 1: P7 -> outer_home
- S10 pad 1: P8 -> ring_top
- S100 pad 1: P8 -> mirror_inner_top
- S101 pad 1: P9 -> mirror_inner_num
- S102 pad 1: P16 -> mirror_outer_thumb
- S103 pad 1: P16 -> mirror_middle_thumb
- S104 pad 1: P16 -> mirror_inner_thumb
- S11 pad 1: P9 -> ring_num
- S12 pad 1: P6 -> middle_bottom
- S13 pad 1: P7 -> middle_home
- S14 pad 1: P8 -> middle_top
- S15 pad 1: P9 -> middle_num
- S16 pad 1: P6 -> index_bottom
- S17 pad 1: P7 -> index_home
- S18 pad 1: P8 -> index_top
- S19 pad 1: P9 -> index_num
- S2 pad 1: P8 -> outer_top
- S20 pad 1: P6 -> inner_bottom
- S21 pad 1: P7 -> inner_home
- S22 pad 1: P8 -> inner_top
- S23 pad 1: P9 -> inner_num
- S24 pad 1: P16 -> outer_thumb
- S25 pad 1: P16 -> middle_thumb
- S26 pad 1: P16 -> inner_thumb
- S27 pad 1: P7 -> mirror_outer_home
- S28 pad 1: P8 -> mirror_outer_top
- S29 pad 1: P9 -> mirror_outer_num
- S3 pad 1: P9 -> outer_num
- S30 pad 1: P6 -> mirror_pinky_bottom
- S31 pad 1: P7 -> mirror_pinky_home
- S32 pad 1: P8 -> mirror_pinky_top
- S33 pad 1: P9 -> mirror_pinky_num
- S34 pad 1: P6 -> mirror_ring_bottom
- S35 pad 1: P7 -> mirror_ring_home
- S36 pad 1: P8 -> mirror_ring_top
- S37 pad 1: P9 -> mirror_ring_num
- S38 pad 1: P6 -> mirror_middle_bottom
- S39 pad 1: P7 -> mirror_middle_home
- S4 pad 1: P6 -> pinky_bottom
- S40 pad 1: P8 -> mirror_middle_top
- S41 pad 1: P9 -> mirror_middle_num
- S42 pad 1: P6 -> mirror_index_bottom
- S43 pad 1: P7 -> mirror_index_home
- S44 pad 1: P8 -> mirror_index_top
- S45 pad 1: P9 -> mirror_index_num
- S46 pad 1: P6 -> mirror_inner_bottom
- S47 pad 1: P7 -> mirror_inner_home
- S48 pad 1: P8 -> mirror_inner_top
- S49 pad 1: P9 -> mirror_inner_num
- S5 pad 1: P7 -> pinky_home
- S50 pad 1: P16 -> mirror_outer_thumb
- S51 pad 1: P16 -> mirror_middle_thumb
- S52 pad 1: P16 -> mirror_inner_thumb
- S53 pad 1: P7 -> outer_home
- S54 pad 1: P8 -> outer_top
- S55 pad 1: P9 -> outer_num
- S56 pad 1: P6 -> pinky_bottom
- S57 pad 1: P7 -> pinky_home
- S58 pad 1: P8 -> pinky_top
- S59 pad 1: P9 -> pinky_num
- S6 pad 1: P8 -> pinky_top
- S60 pad 1: P6 -> ring_bottom
- S61 pad 1: P7 -> ring_home
- S62 pad 1: P8 -> ring_top
- S63 pad 1: P9 -> ring_num
- S64 pad 1: P6 -> middle_bottom
- S65 pad 1: P7 -> middle_home
- S66 pad 1: P8 -> middle_top
- S67 pad 1: P9 -> middle_num
- S68 pad 1: P6 -> index_bottom
- S69 pad 1: P7 -> index_home
- S7 pad 1: P9 -> pinky_num
- S70 pad 1: P8 -> index_top
- S71 pad 1: P9 -> index_num
- S72 pad 1: P6 -> inner_bottom
- S73 pad 1: P7 -> inner_home
- S74 pad 1: P8 -> inner_top
- S75 pad 1: P9 -> inner_num
- S76 pad 1: P16 -> outer_thumb
- S77 pad 1: P16 -> middle_thumb
- S78 pad 1: P16 -> inner_thumb
- S79 pad 1: P7 -> mirror_outer_home
- S8 pad 1: P6 -> ring_bottom
- S80 pad 1: P8 -> mirror_outer_top
- S81 pad 1: P9 -> mirror_outer_num
- S82 pad 1: P6 -> mirror_pinky_bottom
- S83 pad 1: P7 -> mirror_pinky_home
- S84 pad 1: P8 -> mirror_pinky_top
- S85 pad 1: P9 -> mirror_pinky_num
- S86 pad 1: P6 -> mirror_ring_bottom
- S87 pad 1: P7 -> mirror_ring_home
- S88 pad 1: P8 -> mirror_ring_top
- S89 pad 1: P9 -> mirror_ring_num
- S9 pad 1: P7 -> ring_home
- S90 pad 1: P6 -> mirror_middle_bottom
- S91 pad 1: P7 -> mirror_middle_home
- S92 pad 1: P8 -> mirror_middle_top
- S93 pad 1: P9 -> mirror_middle_num
- S94 pad 1: P6 -> mirror_index_bottom
- S95 pad 1: P7 -> mirror_index_home
- S96 pad 1: P8 -> mirror_index_top
- S97 pad 1: P9 -> mirror_index_num
- S98 pad 1: P6 -> mirror_inner_bottom
- S99 pad 1: P7 -> mirror_inner_home
Other:
- board size 295.7 x 128.2 mm -> 278.5 x 124.1 mm

Commit message: feat: flattened out pcb bottom
Other:
- board size 278.5 x 124.1 mm -> 282.9 x 127.1 mm
Changed lines of the file:
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@@
 (fp_text user B- (at -2.25 0 0) (layer F.SilkS) (effects (font (size 0.8 0.8) (thickness 0.15)) ))
         )
-            (gr_line (start 225.09025861660737 195.4636168) (end 199.66628318339258 195.4636168) (angle 90) (layer Edge.Cuts) (width 0.15))
-(gr_line (start 198.56666617667508 195.36199303603308) (end 132.7520332577847 183.09236207331105) (angle 90) (layer Edge.Cuts) (width 0.15))
-(gr_line (start 130.4305833889987 182.12311374606446) (end 89.81087315911333 153.93096060921602) (angle 90) (layer Edge.Cuts) (width 0.15))
-(gr_line (start 88.44012692277174 152.6127227847106) (end 74.34458120410547 133.90730177893874) (angle 90) (layer Edge.Cuts) (width 0.15))
-(gr_line (start 73.19478591207663 129.4613731222214) (end 80.11115872191795 80.24882311879799) (angle 90) (layer Edge.Cuts) (width 0.15))
-(gr_line (start 85.58567374010215 75.10207067449952) (end 129.09846139385073 71.7043350751498) (angle 90) (layer Edge.Cuts) (width 0.15))
-(gr_line (start 129.46370657781426 71.68699059021603) (end 147.5267736987252 71.3803308605907) (angle 90) (layer Edge.Cuts) (width 0.15))
-(gr_line (start 149.45348402400347 71.66370940170549) (end 184.3486989538198 82.80465746055364) (angle 90) (layer Edge.Cuts) (width 0.15))
-(gr_line (start 186.17356107737206 83.08890050000001) (end 238.58298072262792 83.08890050000001) (angle 90) (layer Edge.Cuts) (width 0.15))
-(gr_line (start 240.4078428461802 82.80465746055364) (end 275.30305777599665 71.66370940170545) (angle 90) (layer Edge.Cuts) (width 0.15))
-(gr_line (start 277.22976810127483 71.3803308605907) (end 295.29283522218583 71.68699059021601) (angle 90) (layer Edge.Cuts) (width 0.15))
-(gr_line (start 295.6580804061494 71.7043350751498) (end 339.17086805989777 75.1020706744995) (angle 90) (layer Edge.Cuts) (width 0.15))
-(gr_line (start 344.64538307808203 80.2488231187981) (end 351.5617558879235 129.46137312222208) (angle 90) (layer Edge.Cuts) (width 0.15))
-(gr_line (start 350.4119605958943 133.9073017789391) (end 336.31641487722817 152.61272278471074) (angle 90) (layer Edge.Cuts) (width 0.15))
-(gr_line (start 334.94566864088677 153.93096060921596) (end 294.3259584110012 182.1231137460645) (angle 90) (layer Edge.Cuts) (width 0.15))
-(gr_line (start 292.0045085422152 183.09236207331108) (end 226.1898756233249 195.36199303603308) (angle 90) (layer Edge.Cuts) (width 0.15))
-(gr_arc (start 199.66628318339258 189.4636168) (end 198.56666618339258 195.3619931) (angle -10.560257269957162) (layer Edge.Cuts) (width 0.15))
-(gr_arc (start 133.85165026450218 177.19398583727795) (end 130.43058336450218 182.12311373727795) (angle -24.202368545690234) (layer Edge.Cuts) (width 0.15))
-(gr_arc (start 93.23194003461674 149.00183270042945) (end 88.44012693461674 152.61272280042945) (angle -18.237374897310616) (layer Edge.Cuts) (width 0.15))
-(gr_arc (start 79.13639431595047 130.2964116946576) (end 73.19478591595046 129.4613730946576) (angle -44.99999898331404) (layer Edge.Cuts) (width 0.15))
-(gr_arc (start 86.05276712579176 81.08386169123423) (end 85.58567372579176 75.10207069123423) (angle -77.53506934648001) (layer Edge.Cuts) (width 0.15))
-(gr_arc (start 129.56555477954024 77.68612609188443) (end 129.46370657954023 71.68699059188444) (angle -3.4923055572808153) (layer Edge.Cuts) (width 0.15))
-(gr_arc (start 147.6286219004512 77.37946636225912) (end 149.4534840004512 71.66370936225913) (angle -18.679279058487325) (layer Edge.Cuts) (width 0.15))
-(gr_arc (start 186.17356107737206 77.08890050000001) (end 184.34869897737207 82.8046575) (angle -17.70665365852048) (layer Edge.Cuts) (width 0.15))
-(gr_arc (start 238.58298072262792 77.08890050000001) (end 238.58298072262792 83.08890050000001) (angle -17.706653658520565) (layer Edge.Cuts) (width 0.15))
-(gr_arc (start 277.1279198995489 77.37946636225911) (end 277.2297680995489 71.38033086225911) (angle -18.679279058486458) (layer Edge.Cuts) (width 0.15))
-(gr_arc (start 295.1909870204599 77.68612609188443) (end 295.6580804204599 71.70433509188443) (angle -3.4923055572810853) (layer Edge.Cuts) (width 0.15))
-(gr_arc (start 338.7037746742082 81.08386169123412) (end 344.6453830742082 80.24882309123412) (angle -77.5350693464825) (layer Edge.Cuts) (width 0.15))
-(gr_arc (start 345.6201474840496 130.29641169465822) (end 350.4119605840496 133.90730179465822) (angle -44.99999898331307) (layer Edge.Cuts) (width 0.15))
-(gr_arc (start 331.52460176538324 149.00183270042947) (end 334.94566866538327 153.93096060042947) (angle -18.23737489730803) (layer Edge.Cuts) (width 0.15))
-(gr_arc (start 290.9048915354977 177.19398583727795) (end 292.00450853549773 183.09236213727795) (angle -24.202368545690092) (layer Edge.Cuts) (width 0.15))
-(gr_arc (start 225.09025861660737 189.4636168) (end 225.09025861660737 195.4636168) (angle -10.56025726995739) (layer Edge.Cuts) (width 0.15))
+            (gr_line (start 282.4656211523903 194.99586060000001) (end 142.2909206476096 194.99586060000001) (angle 90) (layer Edge.Cuts) (width 0.15))
+(gr_line (start 139.3064153146483 194.00743487547766) (end 87.45011955354227 155.4277210751701) (angle 90) (layer Edge.Cuts) (width 0.15))
+(gr_line (start 86.44144727465859 154.4252218839736) (end 71.94936302876356 135.19357647760972) (angle 90) (layer Edge.Cuts) (width 0.15))
+(gr_line (start 70.9912003367347 131.4886359208923) (end 78.63502478832638 77.09999867998124) (angle 90) (layer Edge.Cuts) (width 0.15))
+(gr_line (start 82.93837907934977 72.83803055409699) (end 117.97580767920519 68.25865898098938) (angle 90) (layer Edge.Cuts) (width 0.15))
+(gr_line (start 118.53892019032958 68.21721297764142) (end 137.09655487273582 67.90215689131354) (angle 90) (layer Edge.Cuts) (width 0.15))
+(gr_line (start 137.87729384689806 67.95009618910812) (end 159.64649942178815 71.00955851870992) (angle 90) (layer Edge.Cuts) (width 0.15))
+(gr_line (start 160.4713524018777 71.19776797128046) (end 196.05056628742813 82.5570954513033) (angle 90) (layer Edge.Cuts) (width 0.15))
+(gr_line (start 197.57128473995394 82.79396460000001) (end 227.18525706004607 82.79396460000001) (angle 90) (layer Edge.Cuts) (width 0.15))
+(gr_line (start 228.70597551257185 82.5570954513033) (end 264.2851893981221 71.1977679712805) (angle 90) (layer Edge.Cuts) (width 0.15))
+(gr_line (start 265.1100423782116 71.00955851870995) (end 286.87924795310187 67.95009618910814) (angle 90) (layer Edge.Cuts) (width 0.15))
+(gr_line (start 287.6599869272641 67.90215689131355) (end 306.21762160967046 68.21721297764142) (angle 90) (layer Edge.Cuts) (width 0.15))
+(gr_line (start 306.7807341207947 68.25865898098937) (end 341.81816272065 72.83803055409695) (angle 90) (layer Edge.Cuts) (width 0.15))
+(gr_line (start 346.1215170116736 77.09999867998113) (end 353.7653414632652 131.48863592089174) (angle 90) (layer Edge.Cuts) (width 0.15))
+(gr_line (start 352.80717877123664 135.1935764776095) (end 338.3150945253413 154.4252218839738) (angle 90) (layer Edge.Cuts) (width 0.15))
+(gr_line (start 337.30642224645766 155.42772107517015) (end 285.4501264853517 194.00743487547768) (angle 90) (layer Edge.Cuts) (width 0.15))
+(gr_arc (start 142.2909206476096 189.99586060000001) (end 139.3064153476096 194.00743490000002) (angle -36.64827359379882) (layer Edge.Cuts) (width 0.15))
+(gr_arc (start 90.43462488650357 151.41614679969246) (end 86.44144728650357 154.42522189969245) (angle -16.35172711915851) (layer Edge.Cuts) (width 0.15))
+(gr_arc (start 75.94254064060853 132.18450139332856) (end 70.99120034060853 131.48863589332856) (angle -44.99999898331487) (layer Edge.Cuts) (width 0.15))
+(gr_arc (start 83.58636509220021 77.79586415241738) (end 82.93837909220021 72.83803055241738) (angle -74.55368346133184) (layer Edge.Cuts) (width 0.15))
+(gr_arc (start 118.62379369205564 73.21649257930983) (end 118.53892019205564 68.21721297930983) (angle -6.473691442430308) (layer Edge.Cuts) (width 0.15))
+(gr_arc (start 137.18142837446183 72.90143649298196) (end 137.87729387446183 67.95009619298196) (angle -8.972625096238303) (layer Edge.Cuts) (width 0.15))
+(gr_arc (start 158.95063394935192 75.96089882258376) (end 160.47135234935192 71.19776802258376) (angle -9.70665396224895) (layer Edge.Cuts) (width 0.15))
+(gr_arc (start 197.57128473995394 77.79396460000001) (end 196.05056633995395 82.55709540000001) (angle -17.70665365852082) (layer Edge.Cuts) (width 0.15))
+(gr_arc (start 227.18525706004607 77.79396460000001) (end 227.18525706004607 82.79396460000001) (angle -17.70665365852051) (layer Edge.Cuts) (width 0.15))
+(gr_arc (start 265.8059078506479 75.96089882258379) (end 265.11004235064786 71.00955852258379) (angle -9.70665396224804) (layer Edge.Cuts) (width 0.15))
+(gr_arc (start 287.57511342553806 72.90143649298197) (end 287.6599869255381 67.90215689298198) (angle -8.972625096237948) (layer Edge.Cuts) (width 0.15))
+(gr_arc (start 306.1327481079444 73.21649257930984) (end 306.7807341079444 68.25865897930984) (angle -6.47369144242866) (layer Edge.Cuts) (width 0.15))
+(gr_arc (start 341.1701767077997 77.79586415241744) (end 346.12151700779975 77.09999865241744) (angle -74.55368346133213) (layer Edge.Cuts) (width 0.15))
+(gr_arc (start 348.81400115939135 132.184501393328) (end 352.8071787593914 135.19357649332798) (angle -44.99999898331575) (layer Edge.Cuts) (width 0.15))
+(gr_arc (start 334.32191691349624 151.41614679969257) (end 337.30642221349626 155.42772109969258) (angle -16.351727119156806) (layer Edge.Cuts) (width 0.15))
+(gr_arc (start 282.4656211523903 189.99586060000001) (end 282.4656211523903 194.99586060000001) (angle -36.64827359379916) (layer Edge.Cuts) (width 0.15))
 )

Commit message: feat: slightly flatter bottom and slightly tighter choc plates
Parts:
- moved MCU1 4.46 mm to (212.4, 102.1)
Other:
- board size 282.9 x 127.1 mm -> 282.9 x 126 mm
