File: ecad/pcbs/shockboard.kicad_pcb (KiCad board)
At the start: 2 copper layers, 282.9 x 126 mm, 169 parts

Commit message: wip: routing
Parts:
- moved S3 18.2 mm to (96.0, 69.4), turned to -16 degrees
- moved S55 18.2 mm to (96.0, 69.4), turned to -16 degrees
- moved S29 18.2 mm to (340.6, 103.8), turned to 0 degrees
- moved S81 18.2 mm to (340.6, 103.8), turned to 0 degrees
- moved D3 18.1 mm to (94.7, 73.9), turned to -16 degrees
- moved D29 18.1 mm to (340.6, 108.5), turned to 0 degrees
- moved D1 18.1 mm to (84.2, 110.5), turned to -16 degrees
- moved D27 18.1 mm to (340.6, 146.5), turned to 0 degrees
- moved S1 18.0 mm to (85.5, 106.0), turned to -16 degrees
- moved S53 18.0 mm to (85.5, 106.0), turned to -16 degrees
- moved S27 18.0 mm to (340.6, 141.8), turned to 0 degrees
- moved S79 18.0 mm to (340.6, 141.8), turned to 0 degrees
- moved S2 17.9 mm to (90.7, 87.7), turned to -16 degrees
- moved S54 17.9 mm to (90.7, 87.7), turned to -16 degrees
- moved S28 17.9 mm to (340.6, 122.8), turned to 0 degrees
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Routing:
- net P9: track 0.00 -> 241.5 mm
- net P7: track 0.00 -> 227.3 mm
- net P8: track 0.00 -> 221.2 mm
- net P10: track 0.00 -> 165.3 mm
- net P16: track 0.00 -> 164.1 mm
- net P18: track 0.00 -> 142.7 mm
- net P5: track 0.00 -> 140.8 mm
- net P19: track 0.00 -> 140.7 mm
- net P0: track 0.00 -> 139.8 mm
- net P4: track 0.00 -> 139.6 mm
- net P20: track 0.00 -> 138.2 mm
- net P21: track 0.00 -> 116.5 mm
- net P1: track 0.00 -> 116.4 mm
- net P14: track 0.00 -> 115.2 mm
- net P6: track 0.00 -> 75.7 mm
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Other:
- board size 282.9 x 126 mm -> 280.2 x 147.4 mm

Commit message: wip: routing and fill, missing ground plane vias and silkscreen
Parts:
- moved S3 19.6 mm to (88.5, 87.5), turned to -8 degrees
- moved S55 19.6 mm to (88.5, 87.5), turned to -8 degrees
- moved D3 19.5 mm to (87.8, 92.2), turned to -8 degrees
- moved D1 19.4 mm to (82.5, 129.8), turned to -8 degrees
- moved S1 19.3 mm to (83.2, 125.1), turned to -8 degrees
- moved S53 19.3 mm to (83.2, 125.1), turned to -8 degrees
- moved S2 19.3 mm to (85.8, 106.3), turned to -8 degrees
- moved S54 19.3 mm to (85.8, 106.3), turned to -8 degrees
- moved D2 19.2 mm to (85.2, 111.0), turned to -8 degrees
- moved _3 18.1 mm to (97.1, 94.5), turned to -8 degrees
- moved D4 17.3 mm to (98.7, 151.2), turned to -8 degrees
- moved S4 17.2 mm to (99.4, 146.6), turned to -8 degrees
- moved S56 17.2 mm to (99.4, 146.6), turned to -8 degrees
- moved S29 17.1 mm to (335.5, 87.5), turned to 8 degrees
- moved S81 17.1 mm to (335.5, 87.5), turned to 8 degrees
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Routing:
- net P14: track 115.2 -> 551.0 mm, vias 0 -> 3
- net P16: track 164.1 -> 526.9 mm, vias 0 -> 3
- net P10: track 165.3 -> 521.9 mm, vias 0 -> 6
- net P7: track 227.3 -> 467.8 mm, vias 0 -> 4
- net P8: track 221.2 -> 385.4 mm, vias 0 -> 2
- net RAW: track 0.00 -> 123.8 mm, vias 0 -> 1
- net B+: track 0.00 -> 120.2 mm
- net P21: track 116.5 -> 202.7 mm, vias 0 -> 2
- net P6: track 75.7 -> 157.3 mm
- net P1: track 116.4 -> 197.7 mm, vias 0 -> 1
- net P15: track 67.3 -> 147.0 mm, vias 0 -> 1
- net P0: track 139.8 -> 199.9 mm, vias 0 -> 1
- net P9: track 241.5 -> 297.6 mm
- net P20: track 138.2 -> 194.1 mm, vias 0 -> 2
- net P4: track 139.6 -> 178.0 mm, vias 0 -> 2
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- added copper zone on B.Cu, net GND
- added copper zone on F.Cu, net GND
Other:
- board size 280.2 x 147.4 mm -> 282.9 x 126 mm

Commit message: feat: clean up a few traces
Parts:
- moved D48 0.53 mm to (243.9, 117.8)
- moved D38 0.53 mm to (285.9, 143.7)
- moved D14 0.53 mm to (143.7, 106.0)
- moved D19 0.53 mm to (164.4, 94.8)
- moved S39 0.53 mm to (282.6, 120.2)
- moved S44 0.53 mm to (261.9, 109.0)
- moved S59 0.53 mm to (107.5, 90.6)
- moved S7 0.53 mm to (107.5, 90.6)
- moved S91 0.53 mm to (282.6, 120.2)
- moved S96 0.53 mm to (261.9, 109.0)
- moved T1 0.53 mm to (319.3, 74.1)
- moved _4 0.53 mm to (327.0, 95.0)
- moved S10 0.53 mm to (125.1, 101.7)
- moved S103 0.53 mm to (260.7, 168.8)
- moved S38 0.53 mm to (285.3, 139.0)
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Routing:
- net P9: track 297.6 -> 296.2 mm
- net P1: track 197.7 -> 198.8 mm
- net P0: track 199.9 -> 200.6 mm

Commit message: feat: complete board with fab, no silkscreen yet
Parts:
- removed B1: , E73:SW_TACT_ALPS_SKQGABE010
- added RST1: reset_switch_tht_top, ceoloide:reset_switch_tht_top, F.Cu at (198.6, 94.0)
Routing:
- net RST: track 10.2 -> 7.65 mm
- net P16: track 526.9 -> 529.4 mm
- net GND: vias 0 -> 153
