File: ecad/pcbs/shockboard.kicad_pcb (KiCad board)
At the start: 2 copper layers, 282.9 x 126 mm, 169 parts

Commit message: feat: v1 fab files
Routing:
- net P10: track 521.9 -> 522.4 mm
- net GND: vias 153 -> 154
Other:
- rule pad_to_mask_clearance: 0.05 -> 0
- board text added: "JLCJLCJLCJLC"
