File: ergogen/fairyboard_v1/output/pcbs/fairyboard.kicad_pcb (KiCad board)
At the start: 2 copper layers, 279.2 x 130.7 mm, 169 parts

Commit message: feat: modified rotation, thumb cluster, and split distance
Parts:
- moved T1 45.1 mm to (319.3, 84.6), turned to -0.5 degrees
- moved S41 44.5 mm to (278.7, 98.1), turned to 15 degrees
- moved S93 44.5 mm to (278.7, 98.1), turned to 15 degrees
- moved S37 44.4 mm to (297.8, 96.1), turned to 15 degrees
- moved S89 44.4 mm to (297.8, 96.1), turned to 15 degrees
- moved D41 44.1 mm to (279.9, 102.6), turned to 15 degrees
- moved S45 44.1 mm to (261.6, 107.9), turned to 15 degrees
- moved S97 44.1 mm to (261.6, 107.9), turned to 15 degrees
- moved D37 44.0 mm to (299.0, 100.6), turned to 15 degrees
- moved S101 44.0 mm to (243.7, 114.2), turned to 15 degrees
- moved S49 44.0 mm to (243.7, 114.2), turned to 15 degrees
- moved S29 43.9 mm to (337.2, 96.4), turned to 15 degrees
- moved S81 43.9 mm to (337.2, 96.4), turned to 15 degrees
- moved D45 43.7 mm to (262.9, 112.4), turned to 15 degrees
- moved S33 43.6 mm to (318.9, 101.3), turned to 15 degrees
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Other:
- board size 279.2 x 130.7 mm -> 306.4 x 124.7 mm

Commit message: feat: added nice_view
Parts:
- removed OLED1: OLED, lib:OLED_headers
- added DISP1: , ceoloide:display_nice_view, F.Cu at (207.5, 124.4)
Other:
- board size 306.4 x 124.7 mm -> 306.4 x 134.8 mm
Changed lines of the file:
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@@
 (net 73 "P2")
 (net 74 "P3")
-(net 75 "B+")
+(net 75 "DISP1_1")
+(net 76 "DISP1_2")
+(net 77 "DISP1_4")
+(net 78 "DISP1_5")
+(net 79 "B+")
   (net_class Default "This is the default net class."
     (clearance 0.2)
@@
 (add_net "P2")
 (add_net "P3")
+(add_net "DISP1_1")
+(add_net "DISP1_2")
+(add_net "DISP1_4")
+(add_net "DISP1_5")
 (add_net "B+")
   )
@@
         (pad 24 thru_hole circle (at 13.97 -7.62 0) (size 1.7526 1.7526) (drill 1.0922) (layers *.Cu *.SilkS *.Mask) (net 25 "P9"))
       )
-        (module lib:OLED_headers (layer F.Cu)
-        (at 201.4739933 142.786409 90)
-        (fp_text reference "OLED1" (at 0 0) (layer F.SilkS) hide (effects (font (size 1.27 1.27) (thickness 0.15))))
-        (fp_text value OLED (at 0 -7.3) (layer F.Fab) (effects (font (size 1 1) (thickness 0.15))))
-        (pad 4 thru_hole oval (at 1.6 2.18 360) (size 1.7 1.7) (drill 1) (layers *.Cu *.Mask)
-        (net 73 "P2"))
-        (pad 3 thru_hole oval (at 1.6 4.72 360) (size 1.7 1.7) (drill 1) (layers *.Cu *.Mask)
-        (net 74 "P3"))
-        (pad 2 thru_hole oval (at 1.6 7.26 360) (size 1.7 1.7) (drill 1) (layers *.Cu *.Mask)
-        (net 72 "VCC"))
-        (pad 1 thru_hole rect (at 1.6 9.8 360) (size 1.7 1.7) (drill 1) (layers *.Cu *.Mask)
-        (net 70 "GND"))
-        )
+      (module "ceoloide:display_nice_view" (layer F.Cu)
+        (at 207.4739933 124.360409 0)
+        (attr virtual)
+        (fp_text reference "DISP1" (at 0 20 0) (layer F.SilkS) hide
+          (effects (font (size 1 1) (thickness 0.15)))
+        )
+        (fp_text user %R (at 0 20 0) (layer F.Fab)
+          (effects (font (size 1 1) (thickness 0.15)))
+        )
+        (fp_line (start -6.41 15.37) (end -6.41 18.03) (layer F.SilkS) (width 0.12))
+        (fp_line (start 6.41 18.03) (end -6.41 18.03) (layer F.SilkS) (width 0.12))
+        (fp_line (start 6.41 15.37) (end 6.41 18.03) (layer F.SilkS) (width 0.12))
+        (fp_line (start 6.41 15.37) (end -6.41 15.37) (layer F.SilkS) (width 0.12))
+        (fp_line (start 6.88 14.9) (end 6.88 18.45) (layer F.CrtYd) (width 0.15))
+        (fp_line (start 6.88 18.45) (end -6.82 18.45) (layer F.CrtYd) (width 0.15))
+        (fp_line (start -6.82 18.45) (end -6.82 14.9) (layer F.CrtYd) (width 0.15))
+        (fp_line (start -6.82 14.9) (end 6.88 14.9) (layer F.CrtYd) (width 0.15))
+      (pad 1 thru_hole oval (at -5.08 16.7 270) (size 1.7 1.7) (drill 1) (layers *.Cu *.Mask) (net 73 "P2"))
+      (pad 2 thru_hole oval (at -2.54 16.7 270) (size 1.7 1.7) (drill 1) (layers *.Cu *.Mask) (net 74 "P3"))
+      (pad 3 thru_hole oval (at 0 16.7 270) (size 1.7 1.7) (drill 1) (layers *.Cu *.Mask) (net 72 "VCC"))
+      (pad 4 thru_hole oval (at 2.54 16.7 270) (size 1.7 1.7) (drill 1) (layers *.Cu *.Mask) (net 70 "GND"))
+      (pad 5 thru_hole circle (at 5.08 16.7 270) (size 1.7 1.7) (drill 1) (layers *.Cu *.Mask) (net 67 "P1"))
+      (fp_line (start 5.4 13.4) (end 5.4 -11.9) (layer Dwgs.User) (width 0.15))
+      (fp_line (start -5.4 13.4) (end -5.4 -11.9) (layer Dwgs.User) (width 0.15))
+      (fp_line (start 5.4 -11.9) (end -5.4 -11.9) (layer Dwgs.User) (width 0.15))
+      (fp_line (start -5.4 13.4) (end 5.4 13.4) (layer Dwgs.User) (width 0.15))
+      (fp_line (start -7 -18) (end 7 -18) (layer Dwgs.User) (width 0.15))
+      (fp_line (start 7 18) (end -7 18) (layer Dwgs.User) (width 0.15))
+      (fp_line (start -7 18) (end -7 -18) (layer Dwgs.User) (width 0.15))
+      (fp_line (start 7 18) (end 7 -18) (layer Dwgs.User) (width 0.15))
+    )
             (module "ceoloide:reset_switch_tht_top" (layer F.Cu)
                 (at 193.97399329999996 111.2069584 90)
@@
             (pad "" np_thru_hole circle (at -1.5 0) (size 1 1) (drill 0.9) (layers *.Cu *.Mask))
             (pad 1 smd rect (at 2.25 2.075 -0.5) (size 0.9 1.25) (layers F.Cu F.Paste F.Mask) (net 69 "RAW"))
-            (pad 2 smd rect (at -0.75 2.075 -0.5) (size 0.9 1.25) (layers F.Cu F.Paste F.Mask) (net 75 "B+"))
+            (pad 2 smd rect (at -0.75 2.075 -0.5) (size 0.9 1.25) (layers F.Cu F.Paste F.Mask) (net 79 "B+"))
             (pad 3 smd rect (at -2.25 2.075 -0.5) (size 0.9 1.25) (layers F.Cu F.Paste F.Mask))
             (pad "" smd rect (at 3.7 -1.1 -0.5) (size 0.9 0.9) (layers F.Cu F.Paste F.Mask))
@@
         (fp_line (start -1 1.5) (end -1 2.0) (layer F.SilkS) (width 0.15))
         (fp_line (start -1.25 1.75) (end -0.75 1.75) (layer F.SilkS) (width 0.15))
-        (pad 1 thru_hole rect (at -1 0 0) (size 1.2 1.7) (drill 0.75) (layers *.Cu *.Mask) (net 75 "B+"))
+        (pad 1 thru_hole rect (at -1 0 0) (size 1.2 1.7) (drill 0.75) (layers *.Cu *.Mask) (net 79 "B+"))
         (pad 2 thru_hole oval (at 1 0 0) (size 1.2 1.7) (drill 0.75) (layers *.Cu *.Mask) (net 70 "GND"))
     )
@@
       (pad "1" thru_hole circle locked (at 0 -1.65) (size 0.7 0.7) (drill 0.4) (layers *.Cu *.Mask))
     )
-  (gr_line (start 299.95901427827727 206.80021200000002) (end 114.98897232172261 206.80021200000002) (angle 90) (layer Edge.Cuts) (width 0.15))
-(gr_line (start 111.58921122200671 205.46649410753298) (end 67.88977295303735 164.94379546791112) (angle 90) (layer Edge.Cuts) (width 0.15))
-(gr_line (start 66.95940705275326 163.77751336037818) (end 54.937110992756075 142.95428581090016) (angle 90) (layer Edge.Cuts) (width 0.15))
-(gr_line (start 54.43760884945482 139.16019077250274) (end 68.65276492061354 86.10850596970164) (angle 90) (layer Edge.Cuts) (width 0.15))
+  (gr_line (start 244.03807152438083 216.905439) (end 170.90991507561907 216.905439) (angle 90) (layer Edge.Cuts) (width 0.15))
+(gr_line (start 168.60858753626496 216.34434557590816) (end 119.30852311259791 190.7849918122355) (angle 90) (layer Edge.Cuts) (width 0.15))
+(gr_line (start 119.26848649199997 190.76446304836247) (end 68.66226531706232 165.10305652830942) (angle 90) (layer Edge.Cuts) (width 0.15))
+(gr_line (start 66.59342923581853 163.14362118852836) (end 54.937110992756104 142.95428581090022) (angle 90) (layer Edge.Cuts) (width 0.15))
+(gr_line (start 54.437608849454804 139.1601907725028) (end 68.65276492061354 86.10850596970164) (angle 90) (layer Edge.Cuts) (width 0.15))
 (gr_line (start 73.44344606547267 82.40275270808694) (end 108.77779629772431 82.12750355768038) (angle 90) (layer Edge.Cuts) (width 0.15))
 (gr_line (start 109.34176231594849 82.15499267033996) (end 127.79946636351829 84.10389160347599) (angle 90) (layer Edge.Cuts) (width 0.15))
@@
 (gr_line (start 306.17019030227584 82.12750355768038) (end 341.50454053452745 82.40275270808695) (angle 90) (layer Edge.Cuts) (width 0.15))
 (gr_line (start 346.2952216793865 86.10850596970181) (end 360.5103777505451 139.16019077250257) (angle 90) (layer Edge.Cuts) (width 0.15))
-(gr_line (start 360.010875607244 142.95428581090005) (end 347.98857954724673 163.77751336037818) (angle 90) (layer Edge.Cuts) (width 0.15))
-(gr_line (start 347.05821364696266 164.94379546791112) (end 303.35877537799314 205.4664941075331) (angle 90) (layer Edge.Cuts) (width 0.15))
-(gr_arc (start 114.98897232172261 201.80021200000002) (end 111.5892112217226 205.4664941) (angle -42.839909425451935) (layer Edge.Cuts) (width 0.15))
-(gr_arc (start 71.28953405275327 161.27751336037818) (end 66.95940705275326 163.77751336037818) (angle -17.16009046613155) (layer Edge.Cuts) (width 0.15))
-(gr_arc (start 59.26723799275609 140.45428581090016) (end 54.43760879275609 139.16019081090016) (angle -44.999998002132344) (layer Edge.Cuts) (width 0.15))
+(gr_line (start 360.010875607244 142.95428581090005) (end 348.35455736418146 163.1436211885284) (angle 90) (layer Edge.Cuts) (width 0.15))
+(gr_line (start 346.28572128293763 165.10305652830945) (end 295.6795001080055 190.76446304835963) (angle 90) (layer Edge.Cuts) (width 0.15))
+(gr_line (start 295.6394634874076 190.78499181223256) (end 246.33939906373502 216.34434557590816) (angle 90) (layer Edge.Cuts) (width 0.15))
+(gr_arc (start 170.90991507561907 211.905439) (end 168.60858757561905 216.3443456) (angle -27.404241546605448) (layer Edge.Cuts) (width 0.15))
+(gr_arc (start 117.00719557324375 195.22389838814354) (end 119.30852307324375 190.78499178814354) (angle -0.5155824049005417) (layer Edge.Cuts) (width 0.15))
+(gr_arc (start 70.92355623581854 160.64362118852836) (end 66.59342923581853 163.14362118852836) (angle -33.1113407498778) (layer Edge.Cuts) (width 0.15))
+(gr_arc (start 59.2672379927561 140.4542858109002) (end 54.4376087927561 139.1601908109002) (angle -44.99999800213229) (layer Edge.Cuts) (width 0.15))
 (gr_arc (start 73.48239406391478 87.40260100809911) (end 73.44344606391478 82.40275270809911) (angle -74.55368640611167) (layer Edge.Cuts) (width 0.15))
 (gr_arc (start 108.81674429616642 87.1273518576925) (end 109.34176229616642 82.1549926576925) (angle -6.473689922710506) (layer Edge.Cuts) (width 0.15))
@@
 (gr_arc (start 341.4655925360852 87.40260100809908) (end 346.2952217360852 86.10850600809908) (angle -74.5536864061122) (layer Edge.Cuts) (width 0.15))
 (gr_arc (start 355.68074860724386 140.45428581090005) (end 360.01087560724386 142.95428581090005) (angle -44.99999800213243) (layer Edge.Cuts) (width 0.15))
-(gr_arc (start 343.6584525472467 161.27751336037818) (end 347.0582136472467 164.94379546037817) (angle -17.160090466131464) (layer Edge.Cuts) (width 0.15))
-(gr_arc (start 299.95901427827727 201.80021200000004) (end 299.95901427827727 206.80021200000004) (angle -42.83990942545108) (layer Edge.Cuts) (width 0.15))
+(gr_arc (start 344.0244303641814 160.6436211885284) (end 346.2857212641814 165.1030564885284) (angle -33.111340749877854) (layer Edge.Cuts) (width 0.15))
+(gr_arc (start 297.94079102676176 195.2238983881407) (end 295.67950012676175 190.7644630881407) (angle -0.5155824048996465) (layer Edge.Cuts) (width 0.15))
+(gr_arc (start 244.03807152438083 211.905439) (end 244.03807152438083 216.905439) (angle -27.404241546606272) (layer Edge.Cuts) (width 0.15))
 )

Commit message: wip: invert choc hotswap and move diodes
Parts:
- D1, D10, D11, D12, D13, D14, D15, D16, D17, D18, D19, D2, D20, D21, D22, D23, D24, D25, D26, D27, D28, D29, D3, D30, D31, D32, D33, D34, D35, D36, D37, D38, D39, D4, D40, D41, D42, D43, D44, D45, D46, D47, D48, D49, D5, D50, D51, D52, D6, D7, D8, D9: footprint ComboDiode -> SmtDiode
- moved D12 13.8 mm to (119.8, 143.9)
- moved D16 13.8 mm to (136.9, 153.7)
- moved D17 13.8 mm to (141.8, 135.3)
- moved D20 13.8 mm to (154.9, 160.0)
- moved D21 13.8 mm to (159.8, 141.7)
- moved D24 13.8 mm to (131.6, 173.5)
- moved D25 13.8 mm to (149.9, 178.4)
- moved D4 13.8 mm to (79.6, 147.1)
- moved D5 13.8 mm to (84.6, 128.8)
- moved D8 13.8 mm to (100.7, 141.9)
- moved D1 13.8 mm to (66.2, 123.9)
- moved D10 13.8 mm to (110.5, 105.2)
- moved D11 13.8 mm to (115.5, 86.8)
- moved D13 13.8 mm to (124.8, 125.6)
- moved D14 13.8 mm to (129.7, 107.2)
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
Commit message: feat: remove top row and modify thumb cluster
Parts:
- removed D41, D42, D43, D44, D45, D46, D47, D48, D49, D50, D51, D52: , SmtDiode
- removed S100, S101, S102, S103, S104, S81, S82, S83, S84, S85, S86, S87, S88, S89, S90, S91, S92, S93, S94, S95, S96, S97, S98, S99: , PG1350
- S41, S42, S43, S44, S45, S46, S47, S48, S49, S50, S51, S52: footprint MX -> PG1350
- moved S61 239.8 mm to (347.1, 133.1), turned to -165 degrees
- moved S62 230.0 mm to (342.2, 114.7), turned to -165 degrees
- moved S63 224.8 mm to (333.6, 156.4), turned to -165 degrees
- moved S41 213.7 mm to (67.9, 133.1), turned to 165 degrees
- moved S42 209.2 mm to (72.8, 114.7), turned to 165 degrees
- moved S64 207.8 mm to (328.7, 138.0), turned to -165 degrees
- moved S24 200.5 mm to (328.7, 138.0), turned to 15 degrees
- moved S65 198.0 mm to (323.8, 119.7), turned to -165 degrees
- moved D24 195.8 mm to (322.7, 130.8), turned to 15 degrees
- moved S43 190.5 mm to (81.3, 156.4), turned to 165 degrees
- moved S21 186.5 mm to (347.1, 133.1), turned to 15 degrees
- moved S25 185.1 mm to (323.8, 119.7), turned to 15 degrees
- moved S66 184.5 mm to (312.6, 151.1), turned to -165 degrees
- moved D21 181.9 mm to (341.0, 125.9), turned to 15 degrees
- moved S44 180.7 mm to (86.2, 138.0), turned to 165 degrees
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Connections:
- D10 pad 1: P19 -> P20
- D10 pad 2: ring_top -> middle_home
- D11 pad 1: P18 -> P19
- D11 pad 2: ring_num -> middle_top
- D12 pad 2: middle_bottom -> index_bottom
- D13 pad 2: middle_home -> index_home
- D14 pad 2: middle_top -> index_top
- D15 pad 1: P18 -> P21
- D15 pad 2: middle_num -> inner_bottom
- D16 pad 1: P21 -> P20
- D16 pad 2: index_bottom -> inner_home
- D17 pad 1: P20 -> P19
- D17 pad 2: index_home -> inner_top
- D18 pad 1: P19 -> P15
- D18 pad 2: index_top -> outer_thumb
- D19 pad 1: P18 -> P15
- D19 pad 2: index_num -> middle_thumb
- D20 pad 1: P21 -> P15
- D20 pad 2: inner_bottom -> inner_thumb
- D21 pad 1: P20 -> P0
- D21 pad 2: inner_home -> mirror_outer_home
- D22 pad 1: P19 -> P4
- D22 pad 2: inner_top -> mirror_outer_top
- D23 pad 1: P18 -> P1
- D23 pad 2: inner_num -> mirror_pinky_bottom
- D24 pad 1: P15 -> P0
- D24 pad 2: outer_thumb -> mirror_pinky_home
- D25 pad 1: P15 -> P4
- D25 pad 2: middle_thumb -> mirror_pinky_top
- D26 pad 1: P15 -> P1
- D26 pad 2: inner_thumb -> mirror_ring_bottom
- D27 pad 2: mirror_outer_home -> mirror_ring_home
- D28 pad 2: mirror_outer_top -> mirror_ring_top
- D29 pad 1: P5 -> P1
- D29 pad 2: mirror_outer_num -> mirror_middle_bottom
- D3 pad 1: P18 -> P21
- D3 pad 2: outer_num -> pinky_bottom
- D30 pad 1: P1 -> P0
- D30 pad 2: mirror_pinky_bottom -> mirror_middle_home
- D31 pad 1: P0 -> P4
- D31 pad 2: mirror_pinky_home -> mirror_middle_top
- D32 pad 1: P4 -> P1
- D32 pad 2: mirror_pinky_top -> mirror_index_bottom
- D33 pad 1: P5 -> P0
- D33 pad 2: mirror_pinky_num -> mirror_index_home
- D34 pad 1: P1 -> P4
- D34 pad 2: mirror_ring_bottom -> mirror_index_top
- D35 pad 1: P0 -> P1
- D35 pad 2: mirror_ring_home -> mirror_inner_bottom
- D36 pad 1: P4 -> P0
- D36 pad 2: mirror_ring_top -> mirror_inner_home
- D37 pad 1: P5 -> P4
- D37 pad 2: mirror_ring_num -> mirror_inner_top
- D38 pad 1: P1 -> P6
- D38 pad 2: mirror_middle_bottom -> mirror_outer_thumb
- D39 pad 1: P0 -> P6
- D39 pad 2: mirror_middle_home -> mirror_middle_thumb
- D4 pad 1: P21 -> P20
- D4 pad 2: pinky_bottom -> pinky_home
- D40 pad 1: P4 -> P6
- D40 pad 2: mirror_middle_top -> mirror_inner_thumb
- D5 pad 1: P20 -> P19
- D5 pad 2: pinky_home -> pinky_top
- D6 pad 1: P19 -> P21
- D6 pad 2: pinky_top -> ring_bottom
- D7 pad 1: P18 -> P20
- D7 pad 2: pinky_num -> ring_home
- D8 pad 1: P21 -> P19
- D8 pad 2: ring_bottom -> ring_top
- D9 pad 1: P20 -> P21
- D9 pad 2: ring_home -> middle_bottom
- S10 pad 1: P10 -> P7
- S10 pad 2: ring_top -> middle_home
- S11 pad 1: P10 -> P7
- S11 pad 2: ring_num -> middle_top
- S12 pad 1: P7 -> P8
- S12 pad 2: middle_bottom -> index_bottom
- S13 pad 1: P7 -> P8
- S13 pad 2: middle_home -> index_home
- S14 pad 1: P7 -> P8
- S14 pad 2: middle_top -> index_top
- S15 pad 1: P7 -> P9
- S15 pad 2: middle_num -> inner_bottom
- S16 pad 1: P8 -> P9
- S16 pad 2: index_bottom -> inner_home
- S17 pad 1: P8 -> P9
- S17 pad 2: index_home -> inner_top
- S18 pad 1: P8 -> P7
- S18 pad 2: index_top -> outer_thumb
- S19 pad 2: index_num -> middle_thumb
- S20 pad 2: inner_bottom -> inner_thumb
- S21 pad 1: P9 -> P14
- S21 pad 2: inner_home -> mirror_outer_home
- S22 pad 1: P9 -> P14
- S22 pad 2: inner_top -> mirror_outer_top
- S23 pad 1: P9 -> P16
- S23 pad 2: inner_num -> mirror_pinky_bottom
- S24 pad 1: P7 -> P16
- S24 pad 2: outer_thumb -> mirror_pinky_home
- S25 pad 1: P8 -> P16
- S25 pad 2: middle_thumb -> mirror_pinky_top
- S26 pad 1: P9 -> P10
- S26 pad 2: inner_thumb -> mirror_ring_bottom
- S27 pad 1: P14 -> P10
- S27 pad 2: mirror_outer_home -> mirror_ring_home
- S28 pad 1: P14 -> P10
- S28 pad 2: mirror_outer_top -> mirror_ring_top
- S29 pad 1: P14 -> P7
- S29 pad 2: mirror_outer_num -> mirror_middle_bottom
- S3 pad 1: P14 -> P16
- S3 pad 2: outer_num -> pinky_bottom
- S30 pad 1: P16 -> P7
- S30 pad 2: mirror_pinky_bottom -> mirror_middle_home
- S31 pad 1: P16 -> P7
- S31 pad 2: mirror_pinky_home -> mirror_middle_top
- S32 pad 1: P16 -> P8
- S32 pad 2: mirror_pinky_top -> mirror_index_bottom
- S33 pad 1: P16 -> P8
- S33 pad 2: mirror_pinky_num -> mirror_index_home
- S34 pad 1: P10 -> P8
- S34 pad 2: mirror_ring_bottom -> mirror_index_top
- S35 pad 1: P10 -> P9
- S35 pad 2: mirror_ring_home -> mirror_inner_bottom
- S36 pad 1: P10 -> P9
- S36 pad 2: mirror_ring_top -> mirror_inner_home
- S37 pad 1: P10 -> P9
- S37 pad 2: mirror_ring_num -> mirror_inner_top
- S38 pad 2: mirror_middle_bottom -> mirror_outer_thumb
- S39 pad 1: P7 -> P8
- S39 pad 2: mirror_middle_home -> mirror_middle_thumb
- S4 pad 2: pinky_bottom -> pinky_home
- S40 pad 1: P7 -> P9
- S40 pad 2: mirror_middle_top -> mirror_inner_thumb
- S41 pad 1: P7 -> P14
- S41 pad 2: mirror_middle_num -> outer_home
- S42 pad 1: P8 -> P14
- S42 pad 2: mirror_index_bottom -> outer_top
- S43 pad 1: P8 -> P16
- S43 pad 2: mirror_index_home -> pinky_bottom
- S44 pad 1: P8 -> P16
- S44 pad 2: mirror_index_top -> pinky_home
- S45 pad 1: P8 -> P16
- S45 pad 2: mirror_index_num -> pinky_top
- S46 pad 1: P9 -> P10
- S46 pad 2: mirror_inner_bottom -> ring_bottom
- S47 pad 1: P9 -> P10
- S47 pad 2: mirror_inner_home -> ring_home
- S48 pad 1: P9 -> P10
- S48 pad 2: mirror_inner_top -> ring_top
- S49 pad 1: P9 -> P7
- S49 pad 2: mirror_inner_num -> middle_bottom
- S5 pad 2: pinky_home -> pinky_top
- S50 pad 2: mirror_outer_thumb -> middle_home
- S51 pad 1: P8 -> P7
- S51 pad 2: mirror_middle_thumb -> middle_top
- S52 pad 1: P9 -> P8
- S52 pad 2: mirror_inner_thumb -> index_bottom
- S53 pad 1: P14 -> P8
- S53 pad 2: outer_home -> index_home
- S54 pad 1: P14 -> P8
- S54 pad 2: outer_top -> index_top
- S55 pad 1: P14 -> P9
- S55 pad 2: outer_num -> inner_bottom
- S56 pad 1: P16 -> P9
- S56 pad 2: pinky_bottom -> inner_home
- S57 pad 1: P16 -> P9
- S57 pad 2: pinky_home -> inner_top
- S58 pad 1: P16 -> P7
- S58 pad 2: pinky_top -> outer_thumb
- S59 pad 1: P16 -> P8
- S59 pad 2: pinky_num -> middle_thumb
- S6 pad 1: P16 -> P10
- S6 pad 2: pinky_top -> ring_bottom
- S60 pad 1: P10 -> P9
- S60 pad 2: ring_bottom -> inner_thumb
- S61 pad 1: P10 -> P14
- S61 pad 2: ring_home -> mirror_outer_home
- S62 pad 1: P10 -> P14
- S62 pad 2: ring_top -> mirror_outer_top
- S63 pad 1: P10 -> P16
- S63 pad 2: ring_num -> mirror_pinky_bottom
- S64 pad 1: P7 -> P16
- S64 pad 2: middle_bottom -> mirror_pinky_home
- S65 pad 1: P7 -> P16
- S65 pad 2: middle_home -> mirror_pinky_top
- S66 pad 1: P7 -> P10
- S66 pad 2: middle_top -> mirror_ring_bottom
- S67 pad 1: P7 -> P10
- S67 pad 2: middle_num -> mirror_ring_home
- S68 pad 1: P8 -> P10
- S68 pad 2: index_bottom -> mirror_ring_top
- S69 pad 1: P8 -> P7
- S69 pad 2: index_home -> mirror_middle_bottom
- S7 pad 1: P16 -> P10
- S7 pad 2: pinky_num -> ring_home
- S70 pad 1: P8 -> P7
- S70 pad 2: index_top -> mirror_middle_home
- S71 pad 1: P8 -> P7
- S71 pad 2: index_num -> mirror_middle_top
- S72 pad 1: P9 -> P8
- S72 pad 2: inner_bottom -> mirror_index_bottom
- S73 pad 1: P9 -> P8
- S73 pad 2: inner_home -> mirror_index_home
- S74 pad 1: P9 -> P8
- S74 pad 2: inner_top -> mirror_index_top
- S75 pad 2: inner_num -> mirror_inner_bottom
- S76 pad 1: P7 -> P9
- S76 pad 2: outer_thumb -> mirror_inner_home
- S77 pad 1: P8 -> P9
- S77 pad 2: middle_thumb -> mirror_inner_top
- S78 pad 1: P9 -> P7
- S78 pad 2: inner_thumb -> mirror_outer_thumb
- S79 pad 1: P14 -> P8
- S79 pad 2: mirror_outer_home -> mirror_middle_thumb
- S8 pad 2: ring_bottom -> ring_top
- S80 pad 1: P14 -> P9
- S80 pad 2: mirror_outer_top -> mirror_inner_thumb
- S9 pad 1: P10 -> P7
- S9 pad 2: ring_home -> middle_bottom
Other:
- board size 306.4 x 134.8 mm -> 304.9 x 118.5 mm

Commit message: feat: prototyping shape of fairyboard and added key position adjustments to ergogen
Parts:
- moved D20 16.5 mm to (176.6, 193.3), turned to -47 degrees
- moved S20 15.7 mm to (173.1, 202.0), turned to -47 degrees
- moved S60 15.7 mm to (173.1, 202.0), turned to 133 degrees
- moved S19 12.5 mm to (156.3, 188.5), turned to -30.5 degrees
- moved S59 12.5 mm to (156.3, 188.5), turned to 149.5 degrees
- moved S18 12.3 mm to (136.4, 180.4), turned to -14 degrees
- moved S58 12.3 mm to (136.4, 180.4), turned to 166 degrees
- moved D19 12.3 mm to (157.2, 179.2), turned to -30.5 degrees
- moved D18 12.2 mm to (134.6, 171.1), turned to -14 degrees
- moved D40 10.9 mm to (237.9, 199.1), turned to 47 degrees
- moved S40 10.8 mm to (246.8, 202.0), turned to 47 degrees
- moved S80 10.8 mm to (246.8, 202.0), turned to -133 degrees
- moved S39 7.49 mm to (263.6, 188.5), turned to 30.5 degrees
- moved S79 7.49 mm to (263.6, 188.5), turned to -149.5 degrees
- moved D39 7.41 mm to (255.8, 183.2), turned to 30.5 degrees
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Other:
- board size 304.9 x 118.5 mm -> 305.1 x 129.2 mm

Commit message: feat: adjust stagger on outer and inner column
Parts:
- moved D3 2.00 mm to (82.7, 143.8)
- moved D7 2.00 mm to (108.2, 119.7)
- moved D8 2.00 mm to (112.8, 101.3)
- moved S3 2.00 mm to (84.5, 153.0)
- moved S43 2.00 mm to (84.5, 153.0)
- moved S47 2.00 mm to (110.1, 129.0)
- moved S48 2.00 mm to (114.7, 110.5)
- moved S7 2.00 mm to (110.1, 129.0)
- moved S8 2.00 mm to (114.7, 110.5)
- moved _7 2.00 mm to (94.2, 145.6)
- moved D13 2.00 mm to (144.6, 130.9)
- moved D23 2.00 mm to (330.5, 145.7)
- moved D27 2.00 mm to (304.9, 121.7)
- moved D33 2.00 mm to (268.5, 132.8)
- moved D4 2.00 mm to (87.3, 125.3)
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Other:
- board size 305.1 x 129.2 mm -> 306 x 131.1 mm

Commit message: feat: complete fairyboard shape
Other:
- board size 306 x 131.1 mm -> 305.2 x 129.9 mm
