File: ergogen/fairyboard_v1/output/pcbs/fairyboard.kicad_pcb (KiCad board)
At the start: 2 copper layers, 305.2 x 129.9 mm, 133 parts

Commit message: feat: reverse column and row net of inverted chocs
Parts:
- moved JST1 16.0 mm to (225.5, 137.6)
- moved DISP1 12.6 mm to (210.5, 134.1)
- moved MCU1 12.6 mm to (210.5, 133.1)
Connections:
- S41 pad 1: P14 -> outer_home
- S41 pad 2: outer_home -> P14
- S42 pad 1: P14 -> outer_top
- S42 pad 2: outer_top -> P14
- S43 pad 1: P16 -> pinky_bottom
- S43 pad 2: pinky_bottom -> P16
- S44 pad 1: P16 -> pinky_home
- S44 pad 2: pinky_home -> P16
- S45 pad 1: P16 -> pinky_top
- S45 pad 2: pinky_top -> P16
- S46 pad 1: P10 -> ring_bottom
- S46 pad 2: ring_bottom -> P10
- S47 pad 1: P10 -> ring_home
- S47 pad 2: ring_home -> P10
- S48 pad 1: P10 -> ring_top
- S48 pad 2: ring_top -> P10
- S49 pad 1: P7 -> middle_bottom
- S49 pad 2: middle_bottom -> P7
- S50 pad 1: P7 -> middle_home
- S50 pad 2: middle_home -> P7
- S51 pad 1: P7 -> middle_top
- S51 pad 2: middle_top -> P7
- S52 pad 1: P8 -> index_bottom
- S52 pad 2: index_bottom -> P8
- S53 pad 1: P8 -> index_home
- S53 pad 2: index_home -> P8
- S54 pad 1: P8 -> index_top
- S54 pad 2: index_top -> P8
- S55 pad 1: P9 -> inner_bottom
- S55 pad 2: inner_bottom -> P9
- S56 pad 1: P9 -> inner_home
- S56 pad 2: inner_home -> P9
- S57 pad 1: P9 -> inner_top
- S57 pad 2: inner_top -> P9
- S58 pad 1: P7 -> outer_thumb
- S58 pad 2: outer_thumb -> P7
- S59 pad 1: P8 -> middle_thumb
- S59 pad 2: middle_thumb -> P8
- S60 pad 1: P9 -> inner_thumb
- S60 pad 2: inner_thumb -> P9
- S61 pad 1: P14 -> mirror_outer_home
- S61 pad 2: mirror_outer_home -> P14
- S62 pad 1: P14 -> mirror_outer_top
- S62 pad 2: mirror_outer_top -> P14
- S63 pad 1: P16 -> mirror_pinky_bottom
- S63 pad 2: mirror_pinky_bottom -> P16
- S64 pad 1: P16 -> mirror_pinky_home
- S64 pad 2: mirror_pinky_home -> P16
- S65 pad 1: P16 -> mirror_pinky_top
- S65 pad 2: mirror_pinky_top -> P16
- S66 pad 1: P10 -> mirror_ring_bottom
- S66 pad 2: mirror_ring_bottom -> P10
- S67 pad 1: P10 -> mirror_ring_home
- S67 pad 2: mirror_ring_home -> P10
- S68 pad 1: P10 -> mirror_ring_top
- S68 pad 2: mirror_ring_top -> P10
- S69 pad 1: P7 -> mirror_middle_bottom
- S69 pad 2: mirror_middle_bottom -> P7
- S70 pad 1: P7 -> mirror_middle_home
- S70 pad 2: mirror_middle_home -> P7
- S71 pad 1: P7 -> mirror_middle_top
- S71 pad 2: mirror_middle_top -> P7
- S72 pad 1: P8 -> mirror_index_bottom
- S72 pad 2: mirror_index_bottom -> P8
- S73 pad 1: P8 -> mirror_index_home
- S73 pad 2: mirror_index_home -> P8
- S74 pad 1: P8 -> mirror_index_top
- S74 pad 2: mirror_index_top -> P8
- S75 pad 1: P9 -> mirror_inner_bottom
- S75 pad 2: mirror_inner_bottom -> P9
- S76 pad 1: P9 -> mirror_inner_home
- S76 pad 2: mirror_inner_home -> P9
- S77 pad 1: P9 -> mirror_inner_top
- S77 pad 2: mirror_inner_top -> P9
- S78 pad 1: P7 -> mirror_outer_thumb
- S78 pad 2: mirror_outer_thumb -> P7
- S79 pad 1: P8 -> mirror_middle_thumb
- S79 pad 2: mirror_middle_thumb -> P8
- S80 pad 1: P9 -> mirror_inner_thumb
- S80 pad 2: mirror_inner_thumb -> P9
Other:
- board size 305.2 x 129.9 mm -> 305.6 x 118.4 mm

Commit message: feat: vik connector
Parts:
- added VIK_IN1: vik-module-connector-horizontal, vik-module-connector-horizontal, F.Cu at (0.00, 0.00)
Other:
- outline, holes or cut-outs redrawn

Commit message: feat: added reset switch side
Parts:
- RST1: value reset_switch_tht_top -> reset_switch_tht_side; footprint ceoloide:reset_switch_tht_top -> restiveengines:reset_switch_tht_side
- turned RST1 to 0 degrees
Connections:
- RST1 pad 1: RST -> GND
- RST1 pad 2: GND -> RST
Changed lines of the file:
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@@
       (fp_line (start 7 18) (end 7 -18) (layer Dwgs.User) (width 0.15))
     )
-            (module "ceoloide:reset_switch_tht_top" (layer F.Cu)
-                (at 196.9588973 106.6573553 90)
-                (fp_text value "reset_switch_tht_top" (at 0 -2.55 180) (layer F.Fab) (effects (font (size 1 1) (thickness 0.15))))
-                (fp_text reference "RST1" (at 0 2.55 180) (layer F.SilkS) hide (effects (font (size 1 1) (thickness 0.15))))
-                (fp_text user "RST" (at 0 0 90) (layer F.SilkS) (effects (font (size 1 1) (thickness 0.15))))
-                (fp_line (start -3 1.75) (end 3 1.75) (layer F.SilkS) (width 0.15))
-                (fp_line (start 3 1.75) (end 3 1.5) (layer F.SilkS) (width 0.15))
-                (fp_line (start -3 1.75) (end -3 1.5) (layer F.SilkS) (width 0.15))
-                (fp_line (start -3 -1.75) (end -3 -1.5) (layer F.SilkS) (width 0.15))
-                (fp_line (start -3 -1.75) (end 3 -1.75) (layer F.SilkS) (width 0.15))
-                (fp_line (start 3 -1.75) (end 3 -1.5) (layer F.SilkS) (width 0.15))
-                (pad 2 thru_hole circle (at -3.25 0 90) (size 2 2) (drill 1.3) (layers *.Cu *.Mask) (net 56 "GND"))
-                (pad 1 thru_hole circle (at 3.25 0 90) (size 2 2) (drill 1.3) (layers *.Cu *.Mask) (net 57 "RST"))
+            (module "restiveengines:reset_switch_tht_side" (layer F.Cu)
+                (at 196.9588973 106.6573553 0)
+                (fp_text value "reset_switch_tht_side" (at 0 -2.55 0) (layer F.Fab) (effects (font (size 1 1) (thickness 0.15))))
+                (fp_text reference "RST1" (at 0 2.55 90) (layer F.SilkS) hide (effects (font (size 1 1) (thickness 0.15))))
+                (fp_text user "RST" (at 0 0 0) (layer F.SilkS) (effects (font (size 1 1) (thickness 0.15))))
+                (fp_rect (start -3.65 -3.25) (end 3.65 2.25) (width 0.12) (fill none) (layer F.SilkS))
+                (fp_rect (start -1.5 -4.97) (end 1.5 -3.25) (width 0.12) (fill none) (layer Dwgs.User))
+                (pad 1 thru_hole circle (at 2.5 -1.25 0) (size 1.7 1.7) (drill 1) (layers *.Cu *.Mask) (net 56 "GND"))
+                (pad 2 thru_hole circle (at -2.5 -1.25 0) (size 1.7 1.7) (drill 1) (layers *.Cu *.Mask) (net 57 "RST"))
+                (pad "" thru_hole circle (at 3.5 1.25 0) (size 2 2) (drill 1.3) (layers *.Cu *.Mask))
+                (pad "" thru_hole circle (at -3.5 1.25 0) (size 2 2) (drill 1.3) (layers *.Cu *.Mask))
             )
         (module E73:SPDT_C128955 (layer F.Cu)

Commit message: feat: move components onto the board
Parts:
- moved VIK_IN1 238.1 mm to (189.5, 144.1)
- moved T1 100.8 mm to (228.5, 115.7), turned to 0 degrees
- moved RST1 11.4 mm to (192.5, 117.2)
Changed lines of the file:
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@@
     )
             (module "restiveengines:reset_switch_tht_side" (layer F.Cu)
-                (at 196.9588973 106.6573553 0)
+                (at 192.4588973 117.1573553 0)
                 (fp_text value "reset_switch_tht_side" (at 0 -2.55 0) (layer F.Fab) (effects (font (size 1 1) (thickness 0.15))))
                 (fp_text reference "RST1" (at 0 2.55 90) (layer F.SilkS) hide (effects (font (size 1 1) (thickness 0.15))))
@@
             )
         (module E73:SPDT_C128955 (layer F.Cu)
-            (at 327.9637282 99.4414603 -1.5)
+            (at 228.4588973 115.6573553 0)
             (fp_text reference "T1" (at 0 0) (layer F.SilkS) hide (effects (font (size 1.27 1.27) (thickness 0.15))))
             (fp_text value "" (at 0 0) (layer F.SilkS) hide (effects (font (size 1.27 1.27) (thickness 0.15))))
@@
             (pad "" np_thru_hole circle (at 1.5 0) (size 1 1) (drill 0.9) (layers *.Cu *.Mask))
             (pad "" np_thru_hole circle (at -1.5 0) (size 1 1) (drill 0.9) (layers *.Cu *.Mask))
-            (pad 1 smd rect (at 2.25 2.075 -1.5) (size 0.9 1.25) (layers F.Cu F.Paste F.Mask) (net 55 "RAW"))
-            (pad 2 smd rect (at -0.75 2.075 -1.5) (size 0.9 1.25) (layers F.Cu F.Paste F.Mask) (net 67 "B+"))
-            (pad 3 smd rect (at -2.25 2.075 -1.5) (size 0.9 1.25) (layers F.Cu F.Paste F.Mask))
-            (pad "" smd rect (at 3.7 -1.1 -1.5) (size 0.9 0.9) (layers F.Cu F.Paste F.Mask))
-            (pad "" smd rect (at 3.7 1.1 -1.5) (size 0.9 0.9) (layers F.Cu F.Paste F.Mask))
-            (pad "" smd rect (at -3.7 1.1 -1.5) (size 0.9 0.9) (layers F.Cu F.Paste F.Mask))
-            (pad "" smd rect (at -3.7 -1.1 -1.5) (size 0.9 0.9) (layers F.Cu F.Paste F.Mask))
+            (pad 1 smd rect (at 2.25 2.075 0) (size 0.9 1.25) (layers F.Cu F.Paste F.Mask) (net 55 "RAW"))
+            (pad 2 smd rect (at -0.75 2.075 0) (size 0.9 1.25) (layers F.Cu F.Paste F.Mask) (net 67 "B+"))
+            (pad 3 smd rect (at -2.25 2.075 0) (size 0.9 1.25) (layers F.Cu F.Paste F.Mask))
+            (pad "" smd rect (at 3.7 -1.1 0) (size 0.9 0.9) (layers F.Cu F.Paste F.Mask))
+            (pad "" smd rect (at 3.7 1.1 0) (size 0.9 0.9) (layers F.Cu F.Paste F.Mask))
+            (pad "" smd rect (at -3.7 1.1 0) (size 0.9 0.9) (layers F.Cu F.Paste F.Mask))
+            (pad "" smd rect (at -3.7 -1.1 0) (size 0.9 0.9) (layers F.Cu F.Paste F.Mask))
         )
     (module JST_PH_S2B-PH-K_02x2.00mm_Angled (layer F.Cu)
@@
     (module "vik-module-connector-horizontal" (version 20210722) (generator pcbnew)
         (layer "F.Cu")
-        (at 0 0 0)
+        (at 189.4588973 144.1499064 0)
         (fp_text reference "VIK_IN1" (at 5.12 -3.56 unlocked) (layer "F.SilkS") hide
             (effects (font (size 1 1) (thickness 0.15)))

Commit message: feat: create spacerhole and move them to appropriate positions
Parts:
- _1, _2, _3, _4, _5, _6, _7, _8: footprint MountingHole_2.2mm_M2_Pad_Via -> SpacerHole_3.2mm_M2_Pad_Via
- moved _5 3.00 mm to (148.4, 171.7)
- moved _6 3.00 mm to (272.6, 171.7)
- moved _3 2.80 mm to (81.9, 124.0)
- moved _4 2.80 mm to (339.0, 124.0)
- moved _1 2.05 mm to (157.6, 134.9)
- moved _2 2.05 mm to (263.4, 134.9)

Commit message: feat: move diodes
Parts:
- moved D20 16.5 mm to (175.2, 209.7), turned to 43 degrees
- moved D1 16.5 mm to (76.1, 137.2), turned to 76 degrees
- moved D10 16.5 mm to (135.1, 136.0), turned to 76 degrees
- moved D2 16.5 mm to (80.7, 118.8), turned to 76 degrees
- moved D4 16.5 mm to (95.0, 139.9), turned to 76 degrees
- moved D5 16.5 mm to (99.6, 121.4), turned to 76 degrees
- moved D7 16.5 mm to (116.0, 134.3), turned to 76 degrees
- moved D8 16.5 mm to (120.6, 115.9), turned to 76 degrees
- moved D11 16.5 mm to (139.7, 117.5), turned to 76 degrees
- moved D14 16.5 mm to (156.9, 127.0), turned to 76 degrees
- moved D17 16.5 mm to (174.5, 135.0), turned to 76 degrees
- moved D3 16.5 mm to (90.4, 158.3), turned to 76 degrees
- moved D6 16.5 mm to (111.4, 152.7), turned to 76 degrees
- moved D9 16.5 mm to (130.5, 154.4), turned to 76 degrees
- moved D12 16.5 mm to (147.7, 163.9), turned to 76 degrees
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
Commit message: fix: VIK OUT instead of VIK IN
Parts:
- removed VIK_IN1: vik-module-connector-horizontal, vik-module-connector-horizontal
- added VIK_OUT1: vik-keyboard-connector-horizontal, vik-keyboard-connector-horizontal, F.Cu at (189.5, 149.1)
Changed lines of the file:
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@@
         (pad 2 thru_hole oval (at 1 0 0) (size 1.2 1.7) (drill 0.75) (layers *.Cu *.Mask) (net 56 "GND"))
     )
-    (module "vik-module-connector-horizontal" (version 20210722) (generator pcbnew)
+    (module "vik-keyboard-connector-horizontal" (version 20210722) (generator pcbnew)
         (layer "F.Cu")
-        (at 189.4588973 144.1499064 0)
-        (fp_text reference "VIK_IN1" (at 5.12 -3.56 unlocked) (layer "F.SilkS") hide
+        (at 189.4588973 149.1499064 0)
+        (fp_text reference "VIK_OUT1" (at 4.25 -3.5 unlocked) (layer "F.SilkS") hide
             (effects (font (size 1 1) (thickness 0.15)))
         )
-        (fp_text value "vik-module-connector-horizontal" (at 0.1 2.5 unlocked) (layer "F.Fab")
+        (fp_text value "vik-keyboard-connector-horizontal" (at 0.05 5.09 unlocked) (layer "F.Fab")
             (effects (font (size 1 1) (thickness 0.15)))
         )
-        (fp_text user "3v3" (at 3.3 -2.7 unlocked) (layer "F.SilkS")
+        (fp_text user "3v3" (at -5.9 -2.7 unlocked) (layer "F.SilkS")
             (effects (font (size 0.75 0.75) (thickness 0.15)) (justify left bottom))
         )
-        (fp_text user "VIK IN" (at -2.36 -3.42 unlocked) (layer "F.SilkS" knockout)
+        (fp_text user "VIK OUT" (at -3.05 -3.48 unlocked) (layer "F.SilkS" knockout)
             (effects (font (size 1 1) (thickness 0.15)) (justify left bottom))
         )

Commit message: feat: add vik throughhole
Parts:
- added VIK_THROUGHHOLE1: vik-keyboard-throughole, vik-keyboard-throughhole, F.Cu at (189.5, 129.6)
Changed lines of the file:
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@@
         (pad "" smd rect (at -4.55 0.686) (size 1.8 2) (layers "F.Cu" "F.Paste" "F.Mask"))
+    )
+    (module "vik-keyboard-throughhole" (version 20210722) (generator pcbnew)
+        (layer "F.Cu")
+        (at 189.4588973 129.6499064 0)
+        (fp_text reference "VIK_THROUGHHOLE1" (at 1.08 -0.5 unlocked) (layer "F.SilkS") hide
+            (effects (font (size 1 1) (thickness 0.15)))
+        )
+        (fp_text value "vik-keyboard-throughole" (at 2.16 1 unlocked) (layer "F.Fab") hide
+            (effects (font (size 1 1) (thickness 0.15)))
+        )
+        (fp_text user "SDA" (at -1.86 -2.97 90 unlocked) (layer "F.SilkS")
+            (effects (font (size 1 1) (thickness 0.15)) (justify left bottom))
+        )
+        (fp_text user "MISO" (at 8.3 -2.87 90 unlocked) (layer "F.SilkS")
+            (effects (font (size 1 1) (thickness 0.15)) (justify left bottom))
+        )
+        (fp_text user "3.3V" (at -4.4 -2.77 90 unlocked) (layer "F.SilkS")
+            (effects (font (size 1 1) (thickness 0.15)) (justify left bottom))
+        )
+        (fp_text user "MOSI" (at 3.22 6.17 90 unlocked) (layer "F.SilkS")
+            (effects (font (size 1 1) (thickness 0.15)) (justify left bottom))
+        )
+        (fp_text user "SCLK" (at 8.3 6.27 90 unlocked) (layer "F.SilkS")
+            (effects (font (size 1 1) (thickness 0.15)) (justify left bottom))
+        )
+        (fp_text user "SPI CS" (at 5.76 7.67 90 unlocked) (layer "F.SilkS")
+            (effects (font (size 1 1) (thickness 0.15)) (justify left bottom))
+        )
+        (fp_text user "RGB" (at 0.68 -2.97 90 unlocked) (layer "F.SilkS")
+            (effects (font (size 1 1) (thickness 0.15)) (justify left bottom))
+        )
+        (fp_text user "GP AD2" (at 5.76 -2.87 90 unlocked) (layer "F.SilkS")
+            (effects (font (size 1 1) (thickness 0.15)) (justify left bottom))
+        )
+        (fp_text user "5V" (at 0.68 4.97 90 unlocked) (layer "F.SilkS")
+            (effects (font (size 1 1) (thickness 0.15)) (justify left bottom))
+        )
+        (fp_text user "SCL" (at -1.86 5.47 90 unlocked) (layer "F.SilkS")
+            (effects (font (size 1 1) (thickness 0.15)) (justify left bottom))
+        )
+        (fp_text user "GND" (at -4.4 5.67 90 unlocked) (layer "F.SilkS")
+            (effects (font (size 1 1) (thickness 0.15)) (justify left bottom))
+        )
+        (fp_text user "GP AD1" (at 3.22 -2.97 90 unlocked) (layer "F.SilkS")
+            (effects (font (size 1 1) (thickness 0.15)) (justify left bottom))
+        )
+        (fp_text user "VIK OUT" (at -7.02 2.99 90 unlocked) (layer "F.SilkS" knockout)
+            (effects (font (size 1 1) (thickness 0.15)) (justify left bottom))
+        )
+        (pad "1" thru_hole circle (at -5 -1.27) (size 1.5 1.5) (drill 1.1) (layers "*.Cu" "*.Mask") (net 55 "RAW"))
+        (pad "2" thru_hole circle (at -5 1.27) (size 1.5 1.5) (drill 1.1) (layers "*.Cu" "*.Mask") (net 56 "GND"))
+        (pad "3" thru_hole circle (at -2.46 -1.27) (size 1.5 1.5) (drill 1.1) (layers "*.Cu" "*.Mask") (net 52 "P4"))
+        (pad "4" thru_hole circle (at -2.46 1.27) (size 1.5 1.5) (drill 1.1) (layers "*.Cu" "*.Mask") (net 62 "P5"))
+        (pad "5" thru_hole circle (at 0.08 -1.27) (size 1.5 1.5) (drill 1.1) (layers "*.Cu" "*.Mask") (net 54 "P6"))
+        (pad "6" thru_hole circle (at 0.08 1.27) (size 1.5 1.5) (drill 1.1) (layers "*.Cu" "*.Mask") (net 55 "RAW"))
+        (pad "7" thru_hole circle (at 2.62 -1.27) (size 1.5 1.5) (drill 1.1) (layers "*.Cu" "*.Mask") (net 12 "P7"))
+        (pad "8" thru_hole circle (at 2.62 1.27) (size 1.5 1.5) (drill 1.1) (layers "*.Cu" "*.Mask") (net 60 "P2"))
+        (pad "9" thru_hole circle (at 5.16 -1.27) (size 1.5 1.5) (drill 1.1) (layers "*.Cu" "*.Mask") (net 16 "P8"))
+        (pad "10" thru_hole circle (at 5.16 1.27) (size 1.5 1.5) (drill 1.1) (layers "*.Cu" "*.Mask") (net 53 "P1"))
+        (pad "11" thru_hole circle (at 7.7 -1.27) (size 1.5 1.5) (drill 1.1) (layers "*.Cu" "*.Mask") (net 20 "P9"))
+        (pad "12" thru_hole circle (at 7.7 1.27) (size 1.5 1.5) (drill 1.1) (layers "*.Cu" "*.Mask") (net 61 "P3"))
     )
     (module "SpacerHole_3.2mm_M2_Pad_Via" (version 20210722) (generator pcbnew) (layer "F.Cu")
